Commit message: Update color chassis to gray

File: description/robot_core.xacro (robot description, xacro)
@@ -32,4 +32,7 @@
         <color rgba="1 0 0 1"/>
     </material>
+    <material name="gray">
+        <color rgba="0.35 0.35 0.35 1"/>
+    </material>
     <!-- BASE LINK -->
     <link name="base_link">
@@ -55,5 +58,5 @@
                 <box size="${chassis_length} ${chassis_width} ${chassis_height}"/>
             </geometry>
-            <material name="black"/>
+            <material name="gray"/>
         </visual>
         <collision>
